Commit message: 開発環境の移植及び環境依存の解除

File: robots/vmegarover.urdf.xacro (robot description, xacro)
@@ -3,8 +3,8 @@
   <xacro:arg name="gazebo" default="classic" />
   <xacro:arg name="use_ros2_control" default="false" />
-  <xacro:include filename="$(find megarover_samples_ros2)/urdf/body/vbody.urdf.xacro"/>
-  <xacro:include filename="$(find megarover_samples_ros2)/urdf/wheel/vwheel.urdf.xacro"/>
-  <xacro:include filename="$(find megarover_samples_ros2)/urdf/lrf/lrf.urdf.xacro"/>
-  <xacro:include filename="$(find megarover_samples_ros2)/urdf/camera/camera.urdf.xacro"/>
+  <xacro:include filename="$(find megarover_dev)/urdf/body/vbody.urdf.xacro"/>
+  <xacro:include filename="$(find megarover_dev)/urdf/wheel/vwheel.urdf.xacro"/>
+  <xacro:include filename="$(find megarover_dev)/urdf/lrf/lrf.urdf.xacro"/>
+  <xacro:include filename="$(find megarover_dev)/urdf/camera/camera.urdf.xacro"/>
   <!-- =============== Link & Joint =============== -->
   <!-- Base -->
@@ -77,5 +77,5 @@
             <remapping>~/odom:=/odom</remapping>
           </ros>
-          <parameters>$(find megarover_samples_ros2)/config/diff_drive_controller.yaml</parameters>
+          <parameters>$(find megarover_dev)/config/diff_drive_controller.yaml</parameters>
         </plugin>
       </gazebo>
@@ -141,5 +141,5 @@
           filename="ign_ros2_control-system"
           name="ign_ros2_control::IgnitionROS2ControlPlugin">
-          <parameters>$(find megarover_samples_ros2)/config/diff_drive_controller.yaml</parameters>
+          <parameters>$(find megarover_dev)/config/diff_drive_controller.yaml</parameters>
           <ros>
             <remapping>~/cmd_vel_unstamped:=/cmd_vel</remapping>

File: urdf/body/vbody.urdf.xacro (robot description, xacro)
@@ -1,5 +1,5 @@
 <?xml version="1.0"?>
 <robot xmlns:xacro="http://ros.org/wiki/xacro">
-  <xacro:include filename="$(find megarover_samples_ros2)/urdf/body/body.gazebo.xacro"/>
+  <xacro:include filename="$(find megarover_dev)/urdf/body/body.gazebo.xacro"/>
   <xacro:macro name="base_v0" params="parent *joint_origin">
     <joint name="base_link_joint" type="fixed">
@@ -11,10 +11,10 @@
       <visual>
         <geometry>
-          <mesh filename="file://$(find megarover_samples_ros2)/models/vmegarover/meshes/dae/vmega_body.dae"/>
+          <mesh filename="file://$(find megarover_dev)/models/vmegarover/meshes/dae/vmega_body.dae"/>
         </geometry>
       </visual>
       <collision>
         <geometry>
-          <mesh filename="file://$(find megarover_samples_ros2)/models/vmegarover/meshes/stl/vmega_body.stl"/>
+          <mesh filename="file://$(find megarover_dev)/models/vmegarover/meshes/stl/vmega_body.stl"/>
         </geometry>
       </collision>

File: urdf/camera/camera.urdf.xacro (robot description, xacro)
@@ -1,6 +1,6 @@
 <?xml version="1.0"?>
 <robot xmlns:xacro="http://ros.org/wiki/xacro">
-  <xacro:include filename="$(find megarover_samples_ros2)/urdf/common.xacro"/>
-  <xacro:include filename="$(find megarover_samples_ros2)/urdf/camera/camera.gazebo.xacro"/>
+  <xacro:include filename="$(find megarover_dev)/urdf/common.xacro"/>
+  <xacro:include filename="$(find megarover_dev)/urdf/camera/camera.gazebo.xacro"/>
   <xacro:macro name="camera_v0" params="prefix parent *joint_origin">
     <joint name="${prefix}_camera_joint" type="fixed">

File: urdf/lrf/lrf.urdf.xacro (robot description, xacro)
@@ -1,6 +1,6 @@
 <?xml version="1.0"?>
 <robot xmlns:xacro="http://ros.org/wiki/xacro">
-  <xacro:include filename="$(find megarover_samples_ros2)/urdf/common.xacro"/>
-  <xacro:include filename="$(find megarover_samples_ros2)/urdf/lrf/lrf.gazebo.xacro"/>
+  <xacro:include filename="$(find megarover_dev)/urdf/common.xacro"/>
+  <xacro:include filename="$(find megarover_dev)/urdf/lrf/lrf.gazebo.xacro"/>
   <xacro:macro name="lrf_v0" params="prefix parent *joint_origin">
     <joint name="${prefix}_lrf_joint" type="fixed">
@@ -12,10 +12,10 @@
       <visual>
         <geometry>
-          <mesh filename="file://$(find megarover_samples_ros2)/models/vmegarover/meshes/dae/lrf.dae"/>
+          <mesh filename="file://$(find megarover_dev)/models/vmegarover/meshes/dae/lrf.dae"/>
         </geometry>
       </visual>
       <collision>
         <geometry>
-          <mesh filename="file://$(find megarover_samples_ros2)/models/vmegarover/meshes/stl/lrf.stl"/>
+          <mesh filename="file://$(find megarover_dev)/models/vmegarover/meshes/stl/lrf.stl"/>
         </geometry>
       </collision>

File: urdf/wheel/vwheel.urdf.xacro (robot description, xacro)
@@ -1,6 +1,6 @@
 <?xml version="1.0"?>
 <robot xmlns:xacro="http://ros.org/wiki/xacro">
-  <xacro:include filename="$(find megarover_samples_ros2)/urdf/common.xacro"/>
-  <xacro:include filename="$(find megarover_samples_ros2)/urdf/wheel/wheel.gazebo.xacro"/>
+  <xacro:include filename="$(find megarover_dev)/urdf/common.xacro"/>
+  <xacro:include filename="$(find megarover_dev)/urdf/wheel/wheel.gazebo.xacro"/>
   <xacro:property name="wheel_radius" value="0.076"/>
   <xacro:property name="wheel_length" value="0.03"/>
@@ -22,5 +22,5 @@
         </xacro:if>
         <geometry>
-          <mesh filename="file://$(find megarover_samples_ros2)/models/vmegarover/meshes/dae/vmega_wheel.dae"/>
+          <mesh filename="file://$(find megarover_dev)/models/vmegarover/meshes/dae/vmega_wheel.dae"/>
         </geometry>
       </visual>
